Commit message: [Update] add post arm turn in Yaw but not R and P

File: vrx_urdf/wamv_gazebo/urdf/components/wamv_3d_lidar.xacro (robot description, xacro)
@@ -120,5 +120,6 @@
     <xacro:property name="post_to_lidar_x" value="${post_to_post_arm_x+post_arm_to_lidar_x}"/>
     <joint name="${namespace}/base_to_${name}_post_joint" type="fixed">
-      <origin xyz="${x-(post_to_lidar_x)*cos(post_Y)} ${y-(post_to_lidar_x)*sin(post_Y)} ${post_z}" rpy="0 0 ${post_Y}" />
+      <!-- <origin xyz="${x-(post_to_lidar_x)*cos(post_Y)} ${y-(post_to_lidar_x)*sin(post_Y)} ${post_z}" rpy="0 0 ${post_Y}" /> -->
+      <origin xyz="${x} ${y} ${post_z}" rpy="0 0 ${Y}" />
       <parent link="${namespace}/base_link" />
       <child link="${namespace}/${name}_post_link" />
@@ -132,5 +133,6 @@
     <!-- Sensor post arm to lidar joint -->
     <joint name="${namespace}/${name}_post_arm_to_${name}_joint" type="fixed">
-      <origin xyz="${post_arm_to_lidar_x} 0 ${post_arm_to_lidar_z}" rpy="${R} ${P} ${Y-post_Y}" />
+      <!-- <origin xyz="${post_arm_to_lidar_x} 0 ${post_arm_to_lidar_z}" rpy="${R} ${P} ${Y-post_Y}" /> -->
+      <origin xyz="${post_arm_to_lidar_x} 0 ${post_arm_to_lidar_z}" rpy="${R} ${P} 0" />
       <parent link="${namespace}/${name}_post_arm_link" />
       <child link="${namespace}/${name}_link" />

File: vrx_urdf/wamv_gazebo/urdf/components/wamv_camera.xacro (robot description, xacro)
@@ -104,5 +104,6 @@
     <xacro:property name="post_to_camera_x" value="${post_to_post_arm_x+post_arm_to_camera_x}"/>
     <joint name="${namespace}/base_to_${name}_post_joint" type="fixed">
-      <origin xyz="${x-(post_to_camera_x)*cos(post_Y)} ${y-(post_to_camera_x)*sin(post_Y)} ${post_z}" rpy="0 0 ${post_Y}" />
+      <!-- <origin xyz="${x-(post_to_camera_x)*cos(post_Y)} ${y-(post_to_camera_x)*sin(post_Y)} ${post_z}" rpy="0 0 ${post_Y}" /> -->
+      <origin xyz="${x} ${y} ${post_z}" rpy="0 0 ${Y}" />
       <parent link="${namespace}/base_link" />
       <child link="${namespace}/${name}_post_link" />
@@ -116,5 +117,6 @@
     <!-- Sensor post arm to camera joint -->
     <joint name="${namespace}/${name}_post_arm_to_${name}_joint" type="fixed">
-      <origin xyz="${post_arm_to_camera_x} 0 ${post_arm_to_camera_z}" rpy="${R} ${P} ${Y-post_Y}" />
+      <!-- <origin xyz="${post_arm_to_camera_x} 0 ${post_arm_to_camera_z}" rpy="${R} ${P} ${Y-post_Y}" /> -->
+      <origin xyz="${post_arm_to_camera_x} 0 ${post_arm_to_camera_z}" rpy="${R} ${P} 0" />
       <parent link="${namespace}/${name}_post_arm_link" />
       <child link="${namespace}/${name}_link" />
